File: Hardware/Urumi-Nema-17-Node/Urumi-Nema-17-Node.kicad_sch (KiCad schematic)
At the start: 0 parts

Commit message: hw: Basic schematic setup
Parts:
- added C10, C11, C15, C18, C23, C7: 100nF, fab:C_1206, symbol fab:C_1206
- added C12: 10uF, fab:C_1206, symbol fab:C_1206
- added C13, C14: 22pF, Capacitor_SMD:C_0805_2012Metric_Pad1.18x1.45mm_HandSolder, symbol fab:C_1206
- added C16: 220uF, PCM_fab:CP_Elec_100uF_Panasonic_EEE-FN1E101UL, symbol PCM_fab:CP_Elec_100uF_Panasonic_EEE-FN1E101UL
- added C17: 220uF, EEUFS1H221LB:CAPPRD500W60D800H2000, symbol EEUFS1H221LB:EEUFS1H221LB
- added D2: POWER_LED, fab:LED_1206, symbol fab:LED_1206
- added D3: SMD-RGB-HI-LIGHT_6P-L5.0_W5.0_H1.5MM_, SMD-RGB-HI-LIGHT_6P-L5.0_W5.0_H1.5MM_:LED6-SMD-5050, symbol SMD-RGB-HI-LIGHT_6P-L5.0_W5.0_H1.5MM_:SMD-RGB-HI-LIGHT_6P-L5.0_W5.0_H1.5MM_
- added J1, J3: 282814-4, 282814-3:TE_282814-4, symbol 282814-3:282814-4
- added J5: S2B-PH-SM4-TB_LF__SN_, S2B-PH-SM4-TB_LF_SN:JST_S2B-PH-SM4-TB_LF__SN_, symbol S2B-PH-SM4-TB_LF__SN_:S2B-PH-SM4-TB_LF__SN_
- added J6: Conn_02x03_Odd_Even, fab:DIp Switch 3 Position 6 Pin, symbol Connector_Generic:Conn_02x03_Odd_Even
- added J8: PinHeader_01x05_P2.54mm_Horizontal_SMD, fab:PinHeader_01x05_P2.54mm_Horizontal_SMD, symbol fab:PinHeader_01x05_P2.54mm_Horizontal_SMD
- added J9: Thermistor, B2B-XH-A_LF__SN_:JST_B2B-XH-A_LF__SN_, symbol B2B-XH-A_LF__SN_:B2B-XH-A_LF__SN_
- added R10, R11, R5, R9: 1K, fab:R_1206, symbol fab:R_1206
- added R12, R7, R8: 10K, fab:R_1206, symbol fab:R_1206
- added R15: 120, fab:R_1206, symbol fab:R_1206
- added R6: 100K, fab:R_1206, symbol fab:R_1206
- added SW1: Switch_Tactile_CnK, fab:Button_CnK_PTS636.0_6x3.5mm, symbol fab:Switch_Tactile_CnK
- added U1: Microcontroller_AVR128DB32-I_PT, fab:TQFP-32_7x7mm_P0.8mm, symbol fab:Microcontroller_AVR128DB32-I_PT
- added U3: DRV8825_STEPPER_MOTOR_DRIVER_CARRIER, DRV8825 Srepper Motor Driver:IC_DRV8825_STEPPER_MOTOR_DRIVER_CARRIER, symbol DRV8825_STEPPER_MOTOR_DRIVER_CARRIER:DRV8825_STEPPER_MOTOR_DRIVER_CARRIER
- added U5: MAX485E, Package_SO:SOIC-8_3.9x4.9mm_P1.27mm, symbol Interface_UART:MAX485E
- added Y1: 16_MHz_Crystal, 16_MHz-Crystal:H32_RAM, symbol 16_MHz-Crystal:HC49_US-10.244MHZ-16PF-30-EXT-SMD-H32-TR
Connections:
- new net: D3.4 (G+), R11.2
- new net: D3.5 (R+), R9.2
- new net: D3.6 (B+), R10.2
- new net: D2.1 (K), R5.2
- new net A: J1.1, R15.2, U5.6 (A)
- new net A1: J3.4, U3.12 (A1)
- new net A2: J3.3, U3.11 (A2)
- new net B: J1.2, R15.1, U5.7 (B)
- new net B1: J3.2, U3.13 (B1)
- new net B2: J3.1, U3.14 (B2)
- new net BLUE_LED: R10.1, U1.24 (PF4)
- new net DIP1: J6.1 (Pin_1), U1.1 (PA3)
- new net DIP2: J6.3 (Pin_3), U1.32 (PA2)
- new net DIP3: J6.5 (Pin_5), U1.2 (PA4)
- new net DIR: U1.15 (PD5), U3.8 (DIR)
- new net DI/TX2: U1.20 (PF0_(XTAL32K1)), U5.4 (DI)
- new net EN: U1.16 (PD6), U3.1 (~{EN})
- new net FAULT: U3.10 (~{FLT})
- new net GREEN_LED: R11.1, U1.25 (PF5)
- new net LIMIT_SWITCH: J5.1, R7.1, U1.11 (PD1)
- new net PULSE/STEP: U1.14 (PD4)
- new net PWR_12V: C17.P, C18.1, U3.16 (VMOT)
- new net PWR_24V: C16.1, J1.3
- new net PWR_5V: C10.1, C10.2, C11.1, C11.2, C12.1, C12.2, C13.2, C14.2, C15.2, C16.2, C17.N, C18.2, C23.1, C23.2, C7.1, C7.2, D2.2 (A), D3.1 (B-), D3.2 (R-), D3.3 (G-), J1.4, J5.2, J5.S1 (SHIELD), J5.S2 (SHIELD__1), J6.2 (Pin_2), J6.4 (Pin_4), J6.6 (Pin_6), J8.1 (Pin_1), J8.3 (Pin_3), J9.2, R12.1, R5.1, R6.1, R7.2, R8.1, SW1.1, U1.10 (VDDIO2), U1.18 (AVDD), U1.19 (GND), U1.28 (VDD), U1.29 (GND), U3.15 (GND_MOT), U3.5 (~{RST}), U3.6 (~{SLP}), U3.9 (GND), U5.5 (GND), U5.8 (VCC)
- new net RED_LED: R9.1, U1.22 (PF2)
- new net RO/RX2: U1.21 (PF1_(XTAL32K2)), U5.1 (RO)
- new net RST: R8.2, SW1.2, U1.26 (PF6)
- new net RS_EN/XDIR2: R12.2, U1.23 (PF3), U5.2 (~{RE}), U5.3 (DE)
- new net RX1_Debug: J8.4 (Pin_4), U1.7 (PC1)
- new net STEP: U3.7 (STEP)
- new net TX1_Debug: J8.5 (Pin_5), U1.6 (PC0)
- new net Thermistor: C15.1, J9.1, R6.2, U1.12 (PD2)
- new net UPDI: J8.2 (Pin_2), U1.27 (UPDI)
- new net XTAL1: C13.1, U1.30 (PA0_(XTALHF1)), Y1.2
- new net XTAL2: C14.1, U1.31 (PA1_(XTALHF2)), Y1.1
- no-connect marks 0 -> 3
Other:
- added sheet Buck Converter (Buck_Converter.kicad_sch)
- note added: "16 Mhz Crystal"
- note added: "24V Power Input RS485"
- note added: "AVR128DB32 MCU"
- note added: "Bias resistors are not needed in slave nodes, it's only needed in master node."
- note added: "For DRV8825/TMC2130"
- note added: "Limit Switch JST"
- note added: "MAX485E RS485 Module"
- note added: "Motor Out"
- note added: "NODE SELECTION DIP SWITCH"
- note added: "POWER_LED"
- note added: "Place close to MCU"
- note added: "RESET SWITCH"
- note added: "RGB Debug LED"
- note added: "SPI Interface for TMC2130"
- note added: "Stepper Motor Driver Mount for StepStick"
- note added: "THERMISTOR"
- note added: "Termination Resistor"
- note added: "Termination resistor only needed in last node"
- note added: "UPDI Programmer Pins"
