File: Hardware/KiCad/Urumi-Nema-17-Node.kicad_pcb (KiCad board)
At the start: 2 copper layers, 55.4 x 55.4 mm, 63 parts, among them J1 Screw_Terminal_01x02_P3.5mm, J2 Limit Switch, J3 395016004, J4 B4B-XH-A_LF__SN_, J5 B4B-XH-A_LF__SN_, J8 PinHeader_01x05_P2.54mm_Horiz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, M0 SolderJumper_2_Open, M1 SolderJumper_2_Open, M2 SolderJumper_2_Open, Q2 SS8050, SW1 Switch_Tactile_CnK, U1 Microcontroller_AVR128DB32-I_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, U2 TPS54302, U3 DRV8825_STEPPER_MOTOR_DRIVER_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, U4 Regulator_Linear_5.0V_1A_OnSe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, U5 MAX485E, Y1 16_MHz_Crystal

Commit message: hw: v2.2a PCB with in and out terminals, just one debug led- no rgb
Parts:
- removed C19: 220uF, EEUFS1H221LB:CAPPRD500W60D800H2000
- removed D3: SMD-RGB-HI-LIGHT_6P-L5.0_W5.0_H1.5MM_, SMD-RGB-HI-LIGHT_6P-L5.0_W5.0_H1.5MM_:LED6-SMD-5050
- removed J2: Limit Switch, B2B-XH-A_LF__SN_:JST_B2B-XH-A_LF__SN_
- removed R10, R11, R9: 1K, Resistor_SMD:R_0805_2012Metric_Pad1.20x1.40mm_HandSolder
- added C16: 220uF, EEUFS1H221LB:CAPPRD500W60D800H2000, F.Cu at (56.9, 158.0)
- added D1: LED_1206, PCM_fab:LED_1206, F.Cu at (63.2, 163.2)
- added J6: Output, 4 Pin:CONN_SD-39501-001_04P_MOL, F.Cu at (91.0, 171.0)
- added R2: 1k, Resistor_SMD:R_0805_2012Metric_Pad1.20x1.40mm_HandSolder, F.Cu at (86.6, 157.9)
- J1: value Screw_Terminal_01x02_P3.5mm -> B3B-XH-A; footprint fab:TerminalBlock_OnShore_1x02_P3.50mm_Horizontal -> fab:JST_B3B-XH-A
- J3: value 395016004 -> Input
- moved J1 38.8 mm to (103.5, 139.2), turned to 90 degrees
- moved R15 30.3 mm to (95.1, 171.0), turned to -90 degrees
- moved JP1 3.18 mm to (98.6, 140.3)
- moved Y1 0.85 mm to (92.0, 165.1)
- moved C14 0.40 mm to (95.7, 161.3)
- moved C13 0.36 mm to (91.8, 161.4)
- moved JP4 0.24 mm to (95.8, 158.4)
- moved JP5 0.24 mm to (101.2, 158.4)
- moved JP6 0.24 mm to (98.5, 158.4)
- moved J8 0.21 mm to (104.3, 146.2)
- moved C7 0.08 mm to (91.8, 158.5)
Connections:
- J1 pad 1: PWR_24V -> PWR_GND
- J1 pad 2: PWR_GND -> LIMIT_SWITCH
- J3 pad 3: B -> PWR_24V
- J3 pad 4: A -> PWR_GND
- U1 pad 9: unconnected-(U1-PC3-Pad9) -> /DIN
Routing:
- net RED_LED: track 27.0 -> 0.00 mm, vias 2 -> 0
- net Net-(D1-A): track 0.00 -> 26.4 mm
- net BLUE_LED: track 25.5 -> 3.39 mm
- net GREEN_LED: track 19.5 -> 0.00 mm
- net A: track 22.1 -> 34.4 mm
- net PWR_GND: track 132.5 -> 122.3 mm
- net B: track 20.7 -> 28.9 mm
- net PWR_5V: track 143.4 -> 150.7 mm
- net LIMIT_SWITCH: track 15.6 -> 19.1 mm
- net Net-(J8-Pin_3): track 12.1 -> 14.4 mm
- net PWR_24V: track 45.0 -> 42.7 mm
- net Net-(D3-B+): track 1.92 -> 0.00 mm
- net Net-(D3-R+): track 1.45 -> 0.00 mm
- net Net-(D3-G+): track 1.23 -> 0.00 mm
- net XTAL1: track 15.0 -> 15.9 mm
Other:
- board text added: "120"
- board text added: "Debug"
- board text added: "IN"
- board text added: "Motor Out"
- board text added: "OUT"
- board text added: "R"
- board text added: "T"
- board text added: "Th"
- board text removed: "RX"
- board text removed: "TX"

Commit message: hw: v2.2a correct one JST - final V2.2a
Parts:
- turned J4 to 180 degrees
Connections:
- J4 pad 1: A2 -> B2
- J4 pad 2: A1 -> B1
- J4 pad 3: B1 -> A1
- J4 pad 4: B2 -> A2
- U1 pad 9: /DIN -> unconnected-(U1-PC3-Pad9)
Routing:
- net PWR_GND: track 122.3 -> 101.3 mm
- net B1: track 9.19 -> 10.2 mm
- net A1: track 9.62 -> 10.7 mm
- net A2: track 10.1 -> 10.9 mm
