File: Hardware/KiCad/Urumi-Nema-17-Node.kicad_pcb (KiCad board)
At the start: 2 copper layers, 55.4 x 55.4 mm, 63 parts, among them J1 Screw_Terminal_01x02_P3.5mm, J2 B3B-XH-A, J3 395016004, J4 B4B-XH-A_LF__SN_, J5 B4B-XH-A_LF__SN_, J8 PinHeader_01x05_P2.54mm_Horiz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, M0 SolderJumper_2_Open, M1 SolderJumper_2_Open, M2 SolderJumper_2_Open, Q2 SS8050, SW1 Switch_Tactile_CnK, U1 Microcontroller_AVR128DB32-I_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, U2 TPS54302, U3 DRV8825_STEPPER_MOTOR_DRIVER_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, U4 Regulator_Linear_5.0V_1A_OnSe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, U5 MAX485E, Y1 16_MHz_Crystal

Commit message: hw: v1.0.1 added test points
Parts:
- added TP1: TestPoint, TestPoint:TestPoint_Pad_1.0x1.0mm, F.Cu at (59.8, 165.0)
- added TP10: TestPoint, TestPoint:TestPoint_Pad_1.0x1.0mm, F.Cu at (101.7, 165.3)
- added TP11: TestPoint, TestPoint:TestPoint_Pad_1.0x1.0mm, F.Cu at (76.2, 160.6)
- added TP12: TestPoint, TestPoint:TestPoint_Pad_1.0x1.0mm, F.Cu at (83.7, 153.0)
- added TP15: TestPoint, TestPoint:TestPoint_Pad_1.0x1.0mm, F.Cu at (100.2, 153.7)
- added TP16: TestPoint, TestPoint:TestPoint_Pad_1.0x1.0mm, F.Cu at (100.2, 155.8)
- added TP2: TestPoint, TestPoint:TestPoint_Pad_1.0x1.0mm, F.Cu at (83.6, 146.1)
- added TP3: TestPoint, TestPoint:TestPoint_Pad_1.0x1.0mm, F.Cu at (76.2, 162.6)
- added TP4: TestPoint, TestPoint:TestPoint_Pad_1.0x1.0mm, F.Cu at (57.3, 165.0)
- added TP5: TestPoint, TestPoint:TestPoint_Pad_1.0x1.0mm, F.Cu at (64.5, 164.7)
- added TP6: TestPoint, TestPoint:TestPoint_Pad_1.0x1.0mm, F.Cu at (66.5, 164.7)
- added TP7: TestPoint, TestPoint:TestPoint_Pad_1.0x1.0mm, F.Cu at (89.7, 128.1)
- added TP8: TestPoint, TestPoint:TestPoint_Pad_1.0x1.0mm, F.Cu at (100.2, 131.3)
- added TP9: TestPoint, TestPoint:TestPoint_Pad_1.0x1.0mm, F.Cu at (97.4, 135.4)
- moved R15 2.15 mm to (65.5, 166.8)
- moved R5 0.67 mm to (91.7, 139.4)
- moved D2 0.67 mm to (91.7, 134.8)
- moved C15 0.60 mm to (86.7, 128.1)
- moved C17 0.46 mm to (77.0, 137.3)
- moved R6 0.37 mm to (91.7, 130.0)
Routing:
- net PWR_GND: track 112.4 -> 126.7 mm
- net PWR_24V: track 102.5 -> 108.0 mm
- net CS: track 0.00 -> 5.19 mm
- net SDI/MOSI: track 0.00 -> 4.72 mm
- net LIMIT_SWITCH: track 19.0 -> 22.4 mm
- net Thermistor: track 35.9 -> 38.5 mm
- net RS_EN/XDIR2: track 26.8 -> 28.4 mm
- net PWR_5V: track 152.9 -> 154.5 mm
- net DI/TX2: track 27.3 -> 28.8 mm
- net RO/RX2: track 21.0 -> 22.1 mm
- net /DIP3: track 7.09 -> 6.32 mm
- net TX1_Debug: track 10.8 -> 11.4 mm
Other:
- board text added: "24V"
