File: Hardware/KiCad/Buck_Converter.kicad_sch (KiCad schematic)
At the start: 15 parts, among them U2 TPS54302, U4 Regulator_Linear_5.0V_1A_OnSe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

Commit message: hw: v2.2 pcb ready for manufacturing
Parts:
- removed R1: 910k, fab:R_1206, symbol fab:R_1206
- removed R2: 75k, fab:R_1206, symbol fab:R_1206
- removed R3: 100k, fab:R_1206, symbol fab:R_1206
- removed R4: 9.1k, fab:R_1206, symbol fab:R_1206
- added R13: 100K, Resistor_SMD:R_0805_2012Metric_Pad1.20x1.40mm_HandSolder, symbol fab:R_1206
- added R14: 9.1K, Resistor_SMD:R_0805_2012Metric_Pad1.20x1.40mm_HandSolder, symbol fab:R_1206
- added R16: 75K, Resistor_SMD:R_0805_2012Metric_Pad1.20x1.40mm_HandSolder, symbol fab:R_1206
- added R17: 910k, Resistor_SMD:R_0805_2012Metric_Pad1.20x1.40mm_HandSolder, symbol fab:R_1206
- C2, C3: value 0.1uF -> 100nF; footprint fab:C_1206 -> Capacitor_SMD:C_0805_2012Metric_Pad1.18x1.45mm_HandSolder
- C4, C5: footprint fab:C_1206 -> Capacitor_SMD:C_1206_3216Metric_Pad1.33x1.80mm_HandSolder
Connections:
- net PWR_24: now also R17.1
- net PWR_GND: now also R14.2, R16.2
- net V_OUT: now also R13.1
- net EN: now reaches U2.5 (EN)
- net EN: now also R16.1, R17.2
- net at C6.2, U2.4 (FB): now also R13.2, R14.1

Commit message: hw:v1.0.0 connected 24v, reoriented motor out, added 3 pin JST
Changed lines of the file:
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@@
-	)
-	(junction
-		(at 67.31 81.28)
-		(diameter 0)
-		(color 0 0 0 0)
 	)
 	(junction
@@
 	(wire
 		(pts
-			(xy 67.31 81.28) (xy 67.31 86.36)
+			(xy 67.31 76.2) (xy 67.31 86.36)
 		)
 		(stroke
@@
 		(pts
 			(xy 140.97 88.9) (xy 140.97 82.55)
-		)
-		(stroke
-			(width 0)
-			(type default)
-		)
-	)
-	(wire
-		(pts
-			(xy 67.31 76.2) (xy 67.31 81.28)
 		)
 		(stroke
@@
 					(unit 1)
 				)
-			)
-		)
-	)
-	(symbol
-		(lib_id "fab:PWR_FLAG")
-		(at 67.31 81.28 90)
-		(unit 1)
-		(body_style 1)
-		(exclude_from_sim no)
-		(in_bom yes)
-		(on_board yes)
-		(in_pos_files yes)
-		(dnp no)
-		(fields_autoplaced yes)
-		(property "Reference" "#FLG02"
-			(at 67.31 81.28 0)
-			(hide yes)
-			(show_name no)
-			(do_not_autoplace no)
-			(effects
-				(font
-					(size 1.27 1.27)
-				)
-			)
-		)
-		(property "Value" "PWR_FLAG"
-			(at 63.5 81.2799 90)
-			(show_name no)
-			(do_not_autoplace no)
-			(effects
-				(font
-					(size 1.27 1.27)
-				)
-				(justify left)
-			)
-		)
-		(property "Footprint" ""
-			(at 67.31 81.28 0)
-			(hide yes)
-			(show_name no)
-			(do_not_autoplace no)
-			(effects
-				(font
-					(size 1.27 1.27)
-				)
-			)
-		)
-		(property "Datasheet" "~"
-			(at 67.31 81.28 0)
-			(hide yes)
-			(show_name no)
-			(do_not_autoplace no)
-			(effects
-				(font
-					(size 1.27 1.27)
-				)
-			)
-		)
-		(property "Description" "Special symbol for telling ERC where power comes from"
-			(at 67.31 81.28 0)
-			(hide yes)
-			(show_name no)
-			(do_not_autoplace no)
-			(effects
-				(font
-					(size 1.27 1.27)
-				)
-			)
-		)
-		(pin "1"
-		)
-		(instances
-			(project "Urumi-Nema-17-Node"
-				(path "/8685699d-ff1f-485f-8f40-0c2a36cf5da3/d0fcb8b3-02f3-47e4-a852-511c1232bb4a"
-					(reference "#FLG02")
-					(unit 1)
-				)
