File: Hardware/KiCad/Urumi-Nema-17-Node.kicad_sch (KiCad schematic)
At the start: 33 parts, among them J1 282814-4, J3 282814-4, J5 S2B-PH-SM4-TB_LF__SN_, J6 Conn_02x03_Odd_Even, J8 PinHeader_01x05_P2.54mm_Horiz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, J9 Thermistor, SW1 Switch_Tactile_CnK, U1 Microcontroller_AVR128DB32-I_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, U3 DRV8825_STEPPER_MOTOR_DRIVER_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, U5 MAX485E, Y1 16_MHz_Crystal

Commit message: hw: v2.2 pcb ready for manufacturing
Parts:
- removed C16: 220uF, PCM_fab:CP_Elec_100uF_Panasonic_EEE-FN1E101UL, symbol PCM_fab:CP_Elec_100uF_Panasonic_EEE-FN1E101UL
- removed J1, J3: 282814-4, 282814-3:TE_282814-4, symbol 282814-3:282814-4
- removed J5: S2B-PH-SM4-TB_LF__SN_, S2B-PH-SM4-TB_LF_SN:JST_S2B-PH-SM4-TB_LF__SN_, symbol S2B-PH-SM4-TB_LF__SN_:S2B-PH-SM4-TB_LF__SN_
- removed J6: Conn_02x03_Odd_Even, fab:DIp Switch 3 Position 6 Pin, symbol Connector_Generic:Conn_02x03_Odd_Even
- removed J9: Thermistor, B2B-XH-A_LF__SN_:JST_B2B-XH-A_LF__SN_, symbol B2B-XH-A_LF__SN_:B2B-XH-A_LF__SN_
- added C19: 220uF, EEUFS1H221LB:CAPPRD500W60D800H2000, symbol EEUFS1H221LB:EEUFS1H221LB
- added H1, H2, H3, H4: (no value), PCM_fab:MountingHole_M3, symbol PCM_fab:MountingHole_M3
- added J1: Screw_Terminal_01x02_P3.5mm, fab:TerminalBlock_OnShore_1x02_P3.50mm_Horizontal, symbol fab:Screw_Terminal_01x02_P3.5mm
- added J2: Limit Switch, B2B-XH-A_LF__SN_:JST_B2B-XH-A_LF__SN_, symbol B2B-XH-A_LF__SN_:B2B-XH-A_LF__SN_
- added J3: 395016004, 4 Pin:CONN_SD-39501-001_04P_MOL, symbol 395016004:395016004
- added J4, J5: B4B-XH-A_LF__SN_, B4B-XH-A_LF__SN_:JST_B4B-XH-A_LF__SN_, symbol B4B-XH-A_LF__SN_:B4B-XH-A_LF__SN_
- added JP1, JP4, JP5, JP6, M0, M1, M2: SolderJumper_2_Open, Jumper:SolderJumper-2_P1.3mm_Open_Pad1.0x1.5mm, symbol Jumper:SolderJumper_2_Open
- added Laser1: L, B2B-XH-A_LF__SN_:JST_B2B-XH-A_LF__SN_, symbol B2B-XH-A_LF__SN_:B2B-XH-A_LF__SN_
- added Q2: SS8050, Package_TO_SOT_SMD:SOT-23, symbol Transistor_BJT:SS8050
- added R1: 1K, Resistor_SMD:R_0805_2012Metric_Pad1.20x1.40mm_HandSolder, symbol fab:R_1206
- added Thermistor1: Thermistor, B2B-XH-A_LF__SN_:JST_B2B-XH-A_LF__SN_, symbol B2B-XH-A_LF__SN_:B2B-XH-A_LF__SN_
- C10, C11, C15, C18, C23, C7: footprint fab:C_1206 -> Capacitor_SMD:C_0805_2012Metric_Pad1.18x1.45mm_HandSolder
- R10, R11, R12, R15, R5, R6, R7, R8, R9: footprint fab:R_1206 -> Resistor_SMD:R_0805_2012Metric_Pad1.20x1.40mm_HandSolder
- SW1: footprint fab:Button_CnK_PTS636.0_6x3.5mm -> fab:Button_Mini_3.9x3
Connections:
- net STEP is gone; now on net PULSE/STEP: U3.7 (STEP)
- net A: now also J3.2, J3.4
- net A1: now also J4.2
- net A2: now also J4.1
- net B: now also J3.1, J3.3
- net B1: now also J4.3
- net B2: now also J4.4
- net DIP1: now also U1.32 (PA2), JP4.2 (B); no longer U1.1 (PA3)
- net DIP2: now also U1.8 (PC2), JP6.1 (A); no longer U1.32 (PA2)
- net DIP3: now also U1.1 (PA3), JP5.2 (B); no longer U1.2 (PA4)
- net DIR: now also J5.3
- net EN: now also J5.1
- net LIMIT_SWITCH: now also J2.2
- net PULSE/STEP: now also J5.2
- net PWR_24V: now also C19.P, J1.1 (Pin_1)
- net PWR_5V: now also JP1.1 (A), JP4.1 (A), JP5.1 (A), JP6.2 (B), Laser1.1, M0.1 (A), M1.1 (A), M2.1 (A); no longer C10.2, C11.2, C12.2, C13.2, C14.2, C15.2, C17.N, C18.2, C23.1, C7.2, D3.1 (B-), D3.2 (R-), D3.3 (G-), J8.1 (Pin_1), J8.3 (Pin_3), R12.1, R5.1, SW1.1, U1.19 (GND), U1.29 (GND), U3.15 (GND_MOT), U3.9 (GND), U5.5 (GND)
- net Thermistor: now also U1.13 (PD3), Thermistor1.2; no longer U1.12 (PD2)
- net SDO/MISO: now reaches U1.3 (PA5)
- net SCK: now reaches U1.4 (PA6)
- net CS: now reaches U1.5 (PA7)
- net M0: now reaches U3.2 (M0)
- net M0: now also M0.2 (B)
- net M1: now reaches U3.3 (M1)
- net M1: now also M1.2 (B)
- net M2: now reaches U3.4 (M2)
- net M2: now also M2.2 (B)
- new net: Q2.1 (B), R1.2
- new net: J8.3 (Pin_3), JP1.2 (B)
- new net: Laser1.2, Q2.3 (C)
- new net Laser: R1.1, U1.12 (PD2)
- new net PWR_GND: C10.2, C11.2, C12.2, C13.2, C14.2, C15.2, C17.N, C18.2, C19.N, C23.1, C7.2, D3.1 (B-), D3.2 (R-), D3.3 (G-), J1.2 (Pin_2), J2.1, J5.4, J8.1 (Pin_1), Q2.2 (E), R12.1, R5.1, SW1.1, Thermistor1.1, U1.19 (GND), U1.29 (GND), U3.15 (GND_MOT), U3.9 (GND), U5.5 (GND)
- new net SDI/MOSI: U1.2 (PA4)
- no-connect marks 3 -> 2
Other:
- note added: "Interfaces"
- note added: "Laser Module"
- note added: "NEMA 17 Motor Section"
- note removed: "NODE SELECTION DIP SWITCH"
- moved on the sheet: C15, C17, C18, D3, J8, R10, R11, R6, R7, R8, R9, SW1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

Commit message: hw:v1.0.0 connected 24v, reoriented motor out, added 3 pin JST
Parts:
- removed J2: Limit Switch, B2B-XH-A_LF__SN_:JST_B2B-XH-A_LF__SN_, symbol B2B-XH-A_LF__SN_:B2B-XH-A_LF__SN_
- added J2: B3B-XH-A, fab:JST_B3B-XH-A, symbol B3B-XH-A:B3B-XH-A
Connections:
- net PWR_12V is gone; now on net PWR_24V: C17.P, C18.1, U3.16 (VMOT)
- net A1: now also J4.3; no longer J4.2
- net A2: now also J4.4; no longer J4.1
- net B1: now also J4.2; no longer J4.3
- net B2: now also J4.1; no longer J4.4
- net LIMIT_SWITCH: now also J2.2
- net PWR_5V: now also J2.3
- net PWR_GND: now also J2.1

Commit message: hw:v1.0.1 added schematic
Other:
- note added: "DM542 Out"
Changed lines of the file:
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@@
+	)
+	(rectangle
+		(start 198.12 25.4)
+		(end 236.22 85.09)
+		(stroke
+			(width 0)
+			(type default)
+		)
+		(fill
+			(type none)
+		)
 	)
 	(rectangle
@@
 			(font
 				(size 2.54 2.54)
+				(thickness 0.508)
+				(bold yes)
 			)
 		)
@@
 			(font
 				(size 1.27 1.27)
+			)
+		)
+	)
+	(text "DM542 Out"
+		(exclude_from_sim no)
+		(at 217.17 30.48 0)
+		(effects
+			(font
+				(size 2.54 2.54)
+				(thickness 0.508)
+				(bold yes)
 			)
 		)
@@
 			(font
 				(size 2.54 2.54)
-			)
-		)
+				(thickness 0.508)
+				(bold yes)
+			)
+		)

Commit message: hw: v1.0.1 added test points
Parts:
- added TP1, TP10, TP11, TP12, TP15, TP16, TP2, TP3, TP4, TP5, TP6, TP7, TP8, TP9: TestPoint, TestPoint:TestPoint_Pad_1.0x1.0mm, symbol Connector:TestPoint
Connections:
- net A: now also TP5.1
- net B: now also TP6.1
- net CS: now also TP15.1
- net DI/TX2: now also TP12.1
- net LIMIT_SWITCH: now also TP9.1
- net PWR_24V: now also TP1.1
- net PWR_5V: now also TP2.1
- net PWR_GND: now also TP10.1, TP4.1, TP8.1
- net RO/RX2: now also TP11.1
- net RS_EN/XDIR2: now also TP3.1
- net SDI/MOSI: now also TP16.1
- net Thermistor: now also TP7.1
Other:
- note added: "A1324 Hall Effect Sensor needs Analog Input"
- note added: "Limit Switch/Hall Effect JST"
- note removed: "Limit Switch JST"
